Commit message: Change differential driver parametes

File: src/intellwheels_desc/urdf/robot1/base.urdf.xacro (robot description, xacro)
@@ -6,5 +6,5 @@
 		<xacro:property name="dimZ" value="1.00"/> <!-- sem o apoio da cabeca -->
 		<xacro:property name="height" value="0.17"/> <!-- A origem da base.dae esta' no meio dos centros das rodas grandes-->
-		<link name="base_footprint"/>
+		<link name="base_footprint_v2"/>
 		<link name="base_link">
 			<inertial>
@@ -35,5 +35,5 @@
 		</link>
 		<joint name="base_joint" type="fixed">
-			<parent link="base_footprint"/>
+			<parent link="base_footprint_v2"/>
 			<child link="base_link" />
 			<origin xyz="0 0 ${height}"/>

File: src/intellwheels_desc/urdf/robot1/diff_drive.gazebo.xacro (robot description, xacro)
@@ -14,5 +14,5 @@
 				<odometryTopic>odom</odometryTopic>
 				<odometryFrame>odom</odometryFrame>
-				<robotBaseFrame>base_footprint</robotBaseFrame>
+				<robotBaseFrame>base_footprint_v2</robotBaseFrame>
 				<odometrySource>world</odometrySource>
 				<publishWheelTF>false</publishWheelTF>
